File: canbus_transeiver_adapter.kicad_pcb (KiCad board)
At the start: 2 copper layers, 55.6 x 47.8 mm, 17 parts, among them J1 Conn_01x02_Pin, J2 Conn_01x06_Pin, J3 Conn_01x06_Pin, J4 RJ45, J5 Conn_02x03_Odd_Even, J6 Conn_01x06_Socket, U1 LD1117V, U2 MCP2542I/SO

Commit message: Resize a bit
Parts:
- R1, R2: footprint Resistor_THT:R_Axial_DIN0309_L9.0mm_D3.2mm_P2.54mm_Vertical -> Resistor_THT:R_Axial_DIN0309_L9.0mm_D3.2mm_P12.70mm_Horizontal
- moved R1 9.56 mm to (192.3, 135.5), turned to 0 degrees
- moved U1 9.50 mm to (210.3, 139.4), turned to -90 degrees
- moved C1 7.62 mm to (205.6, 145.5)
- moved J1 6.23 mm to (187.8, 139.3), turned to -90 degrees
- moved R2 3.81 mm to (192.3, 139.8), turned to 0 degrees
- moved J2 1.59 mm to (216.9, 108.3)
- moved J6 1.59 mm to (216.9, 145.4)
- moved C2 1.02 mm to (205.6, 151.6)
Routing:
- net Net-(J2-Pin_5): track 80.4 -> 90.8 mm
- net +5V: track 27.6 -> 19.6 mm
- net /+5VCAN: track 36.9 -> 29.6 mm
- net Net-(J2-Pin_6): track 92.6 -> 98.6 mm
- net /CANH: track 96.2 -> 101.4 mm
- net /CANL: track 90.3 -> 94.8 mm
- net /+12CAN: track 97.5 -> 101.8 mm
- net GND: track 282.7 -> 284.6 mm
Other:
- board size 55.6 x 47.8 mm -> 55.6 x 50.9 mm

Commit message: Add a LED on +5V
Parts:
- added D2: LED, LED_THT:LED_D3.0mm, F.Cu at (197.1, 110.7)
- added R5: 330, Resistor_THT:R_Axial_DIN0309_L9.0mm_D3.2mm_P15.24mm_Horizontal, F.Cu at (190.0, 113.2)
- moved R4 3.79 mm to (200.9, 118.4)
- moved C3 2.16 mm to (192.8, 126.9)
- moved C4 2.16 mm to (192.4, 132.4)
- moved U2 2.16 mm to (195.5, 123.2)
Routing:
- net GND: track 284.6 -> 292.0 mm
- net Net-(D2-A): track 0.00 -> 5.57 mm
- net /STBY: track 28.1 -> 31.2 mm
- net /TXD: track 7.58 -> 9.74 mm
- net /VIO: track 16.2 -> 18.4 mm
- net /CANL: track 94.8 -> 92.7 mm
- net /CANH: track 101.4 -> 99.2 mm
- net +5V: track 19.6 -> 21.0 mm
- net /RXD: track 21.3 -> 22.4 mm
